File: NTRIPClient_Hardware/WemosS3_ESP32-S3/KiCad/NTRIPClientBoardWemosS3_ESP32-S3/NTRIPClientBoardWemosS3_ESP32-S3.kicad_pcb (KiCad board)
At the start: 2 copper layers, 68.9 x 133 mm, 19 parts, among them J1 Screw_Terminal_01x04, SW1 RESET, SW2 BUTTON, U1 Wemos_S3_ESP32-S3, U3 BUCK-30V-5V

Commit message: corrected request of mount points so they will be provided when using credentials to the caster Added Atom-Lite M5 to PCB design
Parts:
- added U4: ~, my-KiCad-library:Atom-Lite_M5, F.Cu at (104.8, 139.7)
Routing:
- net /GNSS_RTK_RX: track 11.9 -> 43.2 mm, vias 0 -> 1
- net /5V: track 76.9 -> 104.7 mm
- net /MQTT_PACKET_LED: track 8.99 -> 31.9 mm, vias 0 -> 1
- net /ACQ_RX: track 34.1 -> 55.0 mm
- net /GNSS_RTK_TX: track 11.7 -> 29.7 mm
- net /NTRIP_PACKET_LED: track 14.3 -> 28.3 mm
- net /GND: track 308.1 -> 312.6 mm, vias 229 -> 224
Other:
- board text added: "11-5-2025"
- board text removed: "13-4-2025"
